Commit message: Dataset generation main code ready

File: table/table.urdf (robot description, URDF)
Before this commit: robot table.urdf, 1 links, 0 joints
Links:
- link table: geometry collision mesh filename=/root/ocrtoc_ws/src/rendering_setup_iros22/table/visual/tab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; visual mesh filename=/root/ocrtoc_ws/src/rendering_setup_iros22/table/visual/tab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
